File: projects/07_ais140-2w-gnss-tracker/01_kicad/power_rails.kicad_sch (KiCad schematic)
At the start: 28 parts, among them J2 BATTERY 18650, U3 BQ24074, U4 LC709203F, U5 TLV75733P, U6 TPS22917, U7 TPS22917

Commit message: Project 07: routed 4-layer PCB, fab outputs and 3D for the AIS-140 tracker
- 60x45 mm 4-layer board, double-sided assembly: KiCad DRC 0 errors / 0 unconnected,
  schematic parity clean, ERC clean
- Flow: anchors + greedy placer, GND/+3V3 fan-out, Freerouting 1.9, grid A* finisher
  with rip-up, RF via fences, edge/area stitching, island vias
- Gerbers + drill (zip), JLC BOM/CPL, engineering BOM, assembly PDFs, STEP + renders
  (envelope models for parts without a KiCad 3D model)
- Programming/JTAG via pogo test pads TP21-TP28 + native USB; R12 removed (TMR open)
- Design report updated with layout summary; DRC/ERC report added

Co-Authored-By: Claude Opus 5.5 <noreply@anthropic.com>
Claude-Session: https://claude.ai/code/session_01Hk6s8R6up8HYVQWXd3atVk
Parts:
- removed R12: 46.4k, Resistor_SMD:R_0402_1005Metric, symbol Device:R
- U3: Note EN2=1/EN1=0 -> ILIM resistor mode; CE low = charge enabled -> EN2=1/EN1=0 -> ILIM resistor mode; CE low = charge enabled;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
Connections:
- net CHG_TMR: no longer names the net of U3.14 (TMR)
- no-connect marks 3 -> 4
Other:
- note added: "PART NOTES (VERIFY = check against vendor datasheet before release) U3: EN2=1/EN1=0 -> ILIM resistor mode; CE low = charge enabled; TMR open = default safety timers (VERIFY) R9: IIN_MAX = 1550/R = 1.03 A VERIFY K_ILIM R10: ICHG = 890/R = 500 mA VERIFY K_ISET R11: termination ~10 % ICHG VERIFY R13: fit only when the pack has no NTC R16: VBAT/2 -> ADC1_CH1, 2.1 uA U4: Temperature via I2C (host writ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"
- note removed: "PART NOTES (VERIFY = check against vendor datasheet before release) U3: EN2=1/EN1=0 -> ILIM resistor mode; CE low = charge enabled R9: IIN_MAX = 1550/R = 1.03 A VERIFY K_ILIM R10: ICHG = 890/R = 500 mA VERIFY K_ISET R11: termination ~10 % ICHG VERIFY R12: safety timer VERIFY (open = default timer) R13: fit only when the pack has no NTC R16: VBAT/2 -> ADC1_CH1, 2.1 uA U4: Temperature via I2C (host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"
- moved on the sheet: C14, C15, J2, R13, R14, R15, R16, U4
