File: projects/07_ais140-2w-gnss-tracker/lite/01_kicad/modem.kicad_sch (KiCad schematic)
At the start: 22 parts, among them J4 LTE ANT, Q2 2N7002, U3 EC200U-CN, U8 MFF2 eSIM

Commit message: Tracker 07 Lite (WIP): L-match LTE, passive GNSS patch, bottom test pads, fab script
Co-Authored-By: Claude Opus 5.5 <noreply@anthropic.com>
Claude-Session: https://claude.ai/code/session_01Hk6s8R6up8HYVQWXd3atVk
Parts:
- removed C18: DNP, Capacitor_SMD:C_0402_1005Metric, symbol Device:C
- C19: footprint Capacitor_SMD:C_0402_1005Metric -> Capacitor_SMD:C_0603_1608Metric; MPN 0402 C0G (tune) -> 0603 C0G (tune); Note (none) -> L-match with R14: shunt C or L on the bench
Other:
- note added: "PART NOTES (VERIFY = check against vendor datasheet before release) U3: Runs the tracker firmware (QuecOpen / QuecPython). Land pattern is a reconstruction - VERIFY C16: power-on pulse: tau = C16 x R9 = 2.2 s, PWRKEY low >= 500 ms R10: fit for permanent auto power-on (no PWRKEY shutdown) U8: Pin-out per ETSI TS 102 671 MFF2 (1 GND 2 VPP 3 I/O 6 CLK 7 RST 8 VCC) - VERIFY with the SIM vendor C19: L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"
- note removed: "PART NOTES (VERIFY = check against vendor datasheet before release) U3: Runs the tracker firmware (QuecOpen / QuecPython). Land pattern is a reconstruction - VERIFY C16: power-on pulse: tau = C16 x R9 = 2.2 s, PWRKEY low >= 500 ms R10: fit for permanent auto power-on (no PWRKEY shutdown) U8: Pin-out per ETSI TS 102 671 MFF2 (1 GND 2 VPP 3 I/O 6 CLK 7 RST 8 VCC) - VERIFY with the SIM vendor"
- moved on the sheet: C19, J4, R14
