File: projects/12_multitool-rf-board/01_kicad/crl-mt1.kicad_sch (KiCad schematic)
At the start: 73 parts, among them M1 vibro, SW1 RFswitch, SW2 RFswitch, U1 STM32WB55RG, U10 ESD, U2 CC1101, U3 ST25R3916, U5 ST7565R, U6 BQ25896, U7 BQ27220, U8 LM3281, U8B LM3281, U9 loadsw, X10 BAT+NTC, X6 FFC 18p, Y1 32MHz, Y2 32.768kHz

Commit message: proj12: datasheet-accurate netlist fixes (verified vs KiCad STM32WB55 symbol)
Toward the full fabricable PCB (user chose datasheet-accurate route):
- Complete STM32WB55 power scheme: VDDA/VREF+/VDDRF/VSSRF/VDDUSB, the
  internal SMPS (VDDSMPS/VLXSMPS/VFBSMPS/VSSSMPS) with its 10uH inductor
  (L_SMPS) + 2.2uF VFB decoupling (C_SMPS).
- Fix HSE: 32 MHz crystal now across OSC_IN/OSC_OUT (was wrongly on an
  invented pin with pin2 to GND). All 63 U1 pins now match the official
  KiCad MCU_ST_STM32WB:STM32WB55RGVx symbol exactly (0 missing).
- Fix duplicate designators: LP5562 DA4->DA7, RS3221 DA8 (DA4/DA5 were
  each defined twice, silently merging parts).
- Regenerated schematic (77 parts, 108 nets); ERC still 0 errors.
- Added libsym.py helper for symbol cross-checking.

Approach: use official KiCad symbols for ICs that ship with them (correct
pin-number<->name maps), author the rest from datasheet; next steps are
footprint assignment + placement + routing.

Co-Authored-By: Claude Opus 4.8 <noreply@anthropic.com>
Claude-Session: https://claude.ai/code/session_01Hk6s8R6up8HYVQWXd3atVk
Parts:
- added C_SMPS: 2.2uF, C_0402, symbol crl-mt1:C_SMPS_mcu
- added DA7: LP5562, DSBGA-12, symbol crl-mt1:DA7_io
- added DA8: RS3221-3.3, DFN-6, symbol crl-mt1:DA8_power
- added L_SMPS: 10uH, Inductor_0806, symbol crl-mt1:L_SMPS_mcu
- DA5: value RS3221-3.3 -> LMV331; footprint DFN-6 -> SC-70-5; symbol crl-mt1:DA5_power -> crl-mt1:DA5_rfid125; MPN RS3221-3.3YF3 -> LMV331IDCKR; Manufacturer Runic -> Texas Instruments
Connections:
- net +3V3: now also U1.VDDA, U1.VDDRF, U1.VDDSMPS, U1.VDDUSB, U1.VREF+, DA7.EN, DA7.VDD; no longer DA4.EN, DA4.VDD
- net +3V3_LDO: now also DA8.VOUT; no longer DA5.VOUT
- net GND: now also U1.VSSRF, U1.VSSSMPS, C_SMPS.2, DA7.GND, DA8.GND; no longer DA4.GND, DA5.GND, Y1.2
- net HSE_IN: now also U1.OSC_IN; no longer U1.PB13_OSC
- net I2C_PWR_SCL: now also DA7.SCL; no longer DA4.SCL
- net I2C_PWR_SDA: now also DA7.SDA; no longer DA4.SDA
- net LCD_LED: now also DA7.W; no longer DA4.W
- net LED_B: now also DA7.B; no longer DA4.B
- net LED_G: now also DA7.G; no longer DA4.G
- net LED_R: now also DA7.R; no longer DA4.R
- net VSYS: now also DA8.VIN; no longer DA5.VIN
- new net HSE_OUT: U1.OSC_OUT, Y1.2
- new net SMPS_FB: C_SMPS.1, L_SMPS.2, U1.VFBSMPS
- new net SMPS_LX: L_SMPS.1, U1.VLXSMPS
Other:
- moved on the sheet: ANT1, ANT_LF, ANT_NFC, DA3, D_IR, FLT1, FLT2, J_GPIO, J_IBTN, J_SD, J_SUBG, J_SWD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

Commit message: proj12: transcribe all 8 chip pinouts from datasheets - board complete, 0 pending
Datasheet pads transcribed into pinmap.AUTHORED (with support parts in design.py):
- CC1101 QFN-20 (SWRS061I T19): AVDD x4, GND+EP, +DCOUPL cap
- ST25R3916 UFQFPN-32 (DS12484 Fig4): VDD x8, VSS x6+EP, I2C_EN=GND, AGDC cap,
  SCLK/MISO/MOSI/BSS(SS)/IRQ/RFO1/RFO2/RFI1/RFI2/XTI/XTO mapped exactly
- BQ25896 WQFN-24 (SLUSC76C): +buck inductor, bootstrap, REGN cap, ILIM R, TS divider, CE
- BQ27220 DSBGA-9 (SLUSCB7A): +VDD cap, GPOUT pull-up, BIN pull-down
- LM3281 DSBGA-6 (SNVSA38, was wrongly DSBGA-5): +MODE pin
- LP5562 DSBGA-12 (SNVS820B): +ADDR_SEL0/1, custom 3x4 ball footprint (A1-C4)
- RS3221-3.3 SOT-23-3 (RevA.3, was wrongly DFN-6)

pinmap: multi-pad net support; make_footprints: BGA grid generator.
88 parts, 118 nets, ERC 0 errors; PCB places 87 parts; all pads cross-check clean.

Co-Authored-By: Claude Opus 4.8 <noreply@anthropic.com>
Claude-Session: https://claude.ai/code/session_01Hk6s8R6up8HYVQWXd3atVk
Parts:
- added C_AGDC: 1uF, C_0402, symbol crl-mt1:C_AGDC_nfc
- added C_BTST: 47nF, C_0402, symbol crl-mt1:C_BTST_power
- added C_CCd: 100nF, C_0402, symbol crl-mt1:C_CCd_subghz
- added C_FGV: 2.2uF, C_0402, symbol crl-mt1:C_FGV_power
- added C_REGN: 4.7uF, C_0805, symbol crl-mt1:C_REGN_power
- added L_CHG: 2.2uH, Inductor_0806, symbol crl-mt1:L_CHG_power
- added R_FGB: 10k, R_0402, symbol crl-mt1:R_FGB_power
- added R_FGO: 10k, R_0402, symbol crl-mt1:R_FGO_power
- added R_ILIM: 1.1k, R_0402, symbol crl-mt1:R_ILIM_power
- added R_TS1: 5.23k, R_0402, symbol crl-mt1:R_TS1_power
- added R_TS2: 30.31k, R_0402, symbol crl-mt1:R_TS2_power
- DA8: footprint DFN-6 -> SOT-23
- U8, U8B: footprint DSBGA-5 -> DSBGA-6
Connections:
- net +3V3: no longer U3.VSP
- net GND: now also DA7.ADDR_SEL0, DA7.ADDR_SEL1, U3.I2C_EN, U6.CE, C_AGDC.2, C_CCd.2, C_FGV.2, C_REGN.2, R_FGB.2, R_ILIM.2, R_TS2.2
- net USB_DM: now also U10.I/O1; no longer U10.IO1
- net USB_DP: now also U10.I/O2; no longer U10.IO2
- net VSYS: now also U8.MODE, U8B.MODE, L_CHG.2
- new net CC_DCOUPL: C_CCd.1, U2.DCOUPL
- new net CHG_BTST: C_BTST.2, U6.BTST
- new net CHG_ILIM: R_ILIM.1, U6.ILIM
- new net CHG_REGN: C_REGN.1, R_TS1.1, U6.REGN
- new net CHG_SW: C_BTST.1, L_CHG.1, U6.SW
- new net CHG_TS: R_TS1.2, R_TS2.1, U6.TS
- new net FG_BIN: R_FGB.1, U7.BIN
- new net FG_GPOUT: R_FGO.1, U7.GPOUT
- new net FG_VDD: C_FGV.1, R_FGO.2, U7.VDD
- new net NFC_AGDC: C_AGDC.1, U3.AGDC
Other:
- moved on the sheet: ANT_LF, ANT_NFC, BT1, C1, C10, C2, C3, C4, C5, C6, C7, C8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
