File: projects/12_multitool-rf-board/01_kicad/nova-rf1.kicad_sch (KiCad schematic)
At the start: 88 parts, among them M1 vibro, SW1 RFswitch, SW2 RFswitch, U1 STM32WB55RG, U10 ESD, U2 CC1101, U3 ST25R3916, U5 ST7565R, U6 BQ25896, U7 BQ27220, U8 LM3281, U8B LM3281, U9 loadsw, X10 BAT+NTC, X6 FFC 18p, Y1 32MHz, Y2 32.768kHz

Commit message: proj12: rename board CRL-MT1 -> NOVA-RF1 (project-wide)
Global rename across source, docs, generated schematic/board/footprint-lib,
BOM/CPL, enclosure and fab tooling. No functional change. Footprint library
prefix crl-mt1: -> nova-rf1:; silkscreen/title/fab-file names updated.
(The in-flight compact route output will be renamed when it completes.)

Co-Authored-By: Claude Opus 4.8 <noreply@anthropic.com>
Claude-Session: https://claude.ai/code/session_01Hk6s8R6up8HYVQWXd3atVk
Parts:
- ANT1: symbol crl-mt1:ANT1_mcu -> nova-rf1:ANT1_mcu
- ANT_LF: symbol crl-mt1:ANT_LF_rfid125 -> nova-rf1:ANT_LF_rfid125
- ANT_NFC: symbol crl-mt1:ANT_NFC_nfc -> nova-rf1:ANT_NFC_nfc
- BT1: symbol crl-mt1:BT1_power -> nova-rf1:BT1_power
- C1: symbol crl-mt1:C1_passive -> nova-rf1:C1_passive
- C10: symbol crl-mt1:C10_passive -> nova-rf1:C10_passive
- C2: symbol crl-mt1:C2_passive -> nova-rf1:C2_passive
- C3: symbol crl-mt1:C3_passive -> nova-rf1:C3_passive
- C4: symbol crl-mt1:C4_passive -> nova-rf1:C4_passive
- C5: symbol crl-mt1:C5_passive -> nova-rf1:C5_passive
- C6: symbol crl-mt1:C6_passive -> nova-rf1:C6_passive
- C7: symbol crl-mt1:C7_passive -> nova-rf1:C7_passive
- C8: symbol crl-mt1:C8_passive -> nova-rf1:C8_passive
- C9: symbol crl-mt1:C9_passive -> nova-rf1:C9_passive
- C_AGDC: symbol crl-mt1:C_AGDC_nfc -> nova-rf1:C_AGDC_nfc
- C_BTST: symbol crl-mt1:C_BTST_power -> nova-rf1:C_BTST_power
- C_CCd: symbol crl-mt1:C_CCd_subghz -> nova-rf1:C_CCd_subghz
- C_FGV: symbol crl-mt1:C_FGV_power -> nova-rf1:C_FGV_power
- C_REGN: symbol crl-mt1:C_REGN_power -> nova-rf1:C_REGN_power
- C_SMPS: symbol crl-mt1:C_SMPS_mcu -> nova-rf1:C_SMPS_mcu
- DA3: symbol crl-mt1:DA3_rfid125 -> nova-rf1:DA3_rfid125
- DA4: symbol crl-mt1:DA4_rfid125 -> nova-rf1:DA4_rfid125
- DA5: symbol crl-mt1:DA5_rfid125 -> nova-rf1:DA5_rfid125
- DA7: symbol crl-mt1:DA7_io -> nova-rf1:DA7_io
- DA8: symbol crl-mt1:DA8_power -> nova-rf1:DA8_power
- D_IR: symbol crl-mt1:D_IR_io -> nova-rf1:D_IR_io
- FLT1: symbol crl-mt1:FLT1_mcu -> nova-rf1:FLT1_mcu
- FLT2: symbol crl-mt1:FLT2_subghz -> nova-rf1:FLT2_subghz
- J_GPIO: symbol crl-mt1:J_GPIO_io -> nova-rf1:J_GPIO_io
- J_IBTN: symbol crl-mt1:J_IBTN_io -> nova-rf1:J_IBTN_io
- J_SD: symbol crl-mt1:J_SD_io -> nova-rf1:J_SD_io
- J_SUBG: symbol crl-mt1:J_SUBG_subghz -> nova-rf1:J_SUBG_subghz
- J_SWD: symbol crl-mt1:J_SWD_io -> nova-rf1:J_SWD_io
- J_USB: symbol crl-mt1:J_USB_power -> nova-rf1:J_USB_power
- L13: symbol crl-mt1:L13_power -> nova-rf1:L13_power
- L14: symbol crl-mt1:L14_power -> nova-rf1:L14_power
- LS1: symbol crl-mt1:LS1_ui -> nova-rf1:LS1_ui
- L_CHG: symbol crl-mt1:L_CHG_power -> nova-rf1:L_CHG_power
- L_NFC: symbol crl-mt1:L_NFC_nfc -> nova-rf1:L_NFC_nfc
- L_SMPS: symbol crl-mt1:L_SMPS_mcu -> nova-rf1:L_SMPS_mcu
- M1: symbol crl-mt1:M1_ui -> nova-rf1:M1_ui
- Q_IBTN: symbol crl-mt1:Q_IBTN_io -> nova-rf1:Q_IBTN_io
- Q_IR: symbol crl-mt1:Q_IR_io -> nova-rf1:Q_IR_io
- Q_SPK: symbol crl-mt1:Q_SPK_ui -> nova-rf1:Q_SPK_ui
- Q_VIB: symbol crl-mt1:Q_VIB_ui -> nova-rf1:Q_VIB_ui
- R13: symbol crl-mt1:R13_subghz -> nova-rf1:R13_subghz
- R37: symbol crl-mt1:R37_power -> nova-rf1:R37_power
- RN1: symbol crl-mt1:RN1_io -> nova-rf1:RN1_io
- R_CC1: symbol crl-mt1:R_CC1_power -> nova-rf1:R_CC1_power
- R_CC2: symbol crl-mt1:R_CC2_power -> nova-rf1:R_CC2_power
- R_FGB: symbol crl-mt1:R_FGB_power -> nova-rf1:R_FGB_power
- R_FGO: symbol crl-mt1:R_FGO_power -> nova-rf1:R_FGO_power
- R_ILIM: symbol crl-mt1:R_ILIM_power -> nova-rf1:R_ILIM_power
- R_MID1: symbol crl-mt1:R_MID1_rfid125 -> nova-rf1:R_MID1_rfid125
- R_MID2: symbol crl-mt1:R_MID2_rfid125 -> nova-rf1:R_MID2_rfid125
- R_TS1: symbol crl-mt1:R_TS1_power -> nova-rf1:R_TS1_power
- R_TS2: symbol crl-mt1:R_TS2_power -> nova-rf1:R_TS2_power
- SW1: symbol crl-mt1:SW1_subghz -> nova-rf1:SW1_subghz
- SW2: symbol crl-mt1:SW2_subghz -> nova-rf1:SW2_subghz
- SW_B: symbol crl-mt1:SW_B_ui -> nova-rf1:SW_B_ui
- SW_D: symbol crl-mt1:SW_D_ui -> nova-rf1:SW_D_ui
- SW_L: symbol crl-mt1:SW_L_ui -> nova-rf1:SW_L_ui
- SW_O: symbol crl-mt1:SW_O_ui -> nova-rf1:SW_O_ui
- SW_R: symbol crl-mt1:SW_R_ui -> nova-rf1:SW_R_ui
- SW_U: symbol crl-mt1:SW_U_ui -> nova-rf1:SW_U_ui
- U1: symbol crl-mt1:U1_mcu -> nova-rf1:U1_mcu
- U10: symbol crl-mt1:U10_power -> nova-rf1:U10_power
- U2: symbol crl-mt1:U2_subghz -> nova-rf1:U2_subghz
- U3: symbol crl-mt1:U3_nfc -> nova-rf1:U3_nfc
- U5: symbol crl-mt1:U5_io -> nova-rf1:U5_io
- U6: symbol crl-mt1:U6_power -> nova-rf1:U6_power
- U7: symbol crl-mt1:U7_power -> nova-rf1:U7_power
- U8: symbol crl-mt1:U8_power -> nova-rf1:U8_power
- U8B: symbol crl-mt1:U8B_power -> nova-rf1:U8B_power
- U9: symbol crl-mt1:U9_power -> nova-rf1:U9_power
- U_IR: symbol crl-mt1:U_IR_io -> nova-rf1:U_IR_io
- VD4: symbol crl-mt1:VD4_io -> nova-rf1:VD4_io
- VD_IBTN: symbol crl-mt1:VD_IBTN_io -> nova-rf1:VD_IBTN_io
- VD_USB: symbol crl-mt1:VD_USB_io -> nova-rf1:VD_USB_io
- VT4: symbol crl-mt1:VT4_rfid125 -> nova-rf1:VT4_rfid125
- VT6: symbol crl-mt1:VT6_rfid125 -> nova-rf1:VT6_rfid125
- X10: symbol crl-mt1:X10_power -> nova-rf1:X10_power
- X6: symbol crl-mt1:X6_io -> nova-rf1:X6_io
- X_NFC1: symbol crl-mt1:X_NFC1_nfc -> nova-rf1:X_NFC1_nfc
- Y1: symbol crl-mt1:Y1_mcu -> nova-rf1:Y1_mcu
- Y2: symbol crl-mt1:Y2_mcu -> nova-rf1:Y2_mcu
- ZQ1: symbol crl-mt1:ZQ1_nfc -> nova-rf1:ZQ1_nfc
- ZQ3: symbol crl-mt1:ZQ3_subghz -> nova-rf1:ZQ3_subghz
Other:
- title: CRL-MT1 multi-tool RF board -> NOVA-RF1 multi-tool RF board

Commit message: proj12: level-1 design verification + fix 3 netlist bugs it caught
verify_design.py: firmware pin-map (38/38 vs Flipper F7), power+GND per IC,
decoupling, net sanity -> 32 PASS / 0 FAIL. ERC 0 errors.
Fixed: analog rail +3V3_LDO/A3V3 net-name split (op-amp rail wasn't driven);
125kHz coil driver +5V had no source (-> VSYS); added C_A3V3 decoupling.
04_docs/VERIFICATION.md documents results + how to self-check + bring-up steps.

Co-Authored-By: Claude Opus 4.8 <noreply@anthropic.com>
Claude-Session: https://claude.ai/code/session_01Hk6s8R6up8HYVQWXd3atVk
Parts:
- added C_A3V3: 1uF, C_0402, symbol nova-rf1:C_A3V3_power
Connections:
- net +3V3_LDO is gone; now on net A3V3: DA8.VOUT
- net +5V is gone; now on net VSYS: VT4.S
- net A3V3: now also C_A3V3.1
- net GND: now also C_A3V3.2
Other:
- moved on the sheet: C1, C10, C2, C3, C4, C5, C6, C7, C8, C9, R37, R_CC1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
